File: Hardware/Block_Template.brd (EAGLE design)
At the start: 30.5 x 44.5 mm, 11 parts, among them J1 EDISON_CONNECTOR_FULLMOUNTING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, J2 EDISON_CONNECTOR_FULLHEADER

Commit message: initial cut
Parts:
- removed FID1, FID2, FID3, FID4: FIDUCIAL1X2, SparkFun-Aesthetics:FIDUCIAL-1X2
- removed FRAME1: FRAME-LETTER, SparkFun-Aesthetics:CREATIVE_COMMONS
- removed LOGO1, LOGO2: OSHW-LOGOS, SparkFun-Aesthetics:OSHW-LOGO-S
- removed LOGO3, LOGO4: SFE_LOGO_NAME_FLAME.1_INCH, SparkFun-Aesthetics:SFE_LOGO_NAME_FLAME_.1
Other:
- board size 30.5 x 44.5 mm -> 41.7 x 35.6 mm
- board text removed: "Engineer"
- board text removed: "LEDs & User Switches/Buttons go here"
- board text removed: "Max Board Length"
- board text removed: "Name of Block"
- board text removed: "Note: Units are in Inches"
- board text removed: "Nothing goes here... I mean it."
- board text removed: "User Interface/Connectors"
Changed lines of the file:
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@@
 <?xml version="1.0" encoding="utf-8"?>
 <!DOCTYPE eagle SYSTEM "eagle.dtd">
-<eagle version="6.5.0">
+<eagle version="7.3.0">
 <drawing>
 <settings>
@@
 <board>
 <plain>
-<wire x1="30.48" y1="42.672" x2="30.48" y2="1.778" width="0.1524" layer="20"/>
-<wire x1="28.702" y1="0" x2="1.778" y2="0" width="0.1524" layer="20"/>
-<wire x1="0" y1="1.778" x2="0" y2="42.672" width="0.1524" layer="20"/>
-<text x="29.21" y="-13.97" size="1.6764" layer="51" ratio="15">Engineer</text>
-<hole x="28.575" y="1.905" drill="2"/>
-<hole x="1.905" y="1.905" drill="2"/>
-<hole x="1.905" y="42.545" drill="2"/>
-<hole x="28.575" y="42.545" drill="2"/>
-<text x="15.24" y="45.085" size="1.27" layer="51" align="bottom-center">User Interface/Connectors</text>
-<text x="-0.635" y="22.225" size="1.27" layer="51" rot="R270" align="top-center">LEDs &amp; User Switches/Buttons go here</text>
-<text x="31.115" y="22.225" size="1.27" layer="51" rot="R270" align="bottom-center">Nothing goes here...  I mean it.</text>
-<text x="29.972" y="26.416" size="1.27" layer="21" font="vector" ratio="15" rot="R90">Name of Block</text>
-<wire x1="1.778" y1="44.45" x2="28.702" y2="44.45" width="0.1524" layer="20"/>
-<wire x1="30.48" y1="46.99" x2="30.48" y2="53.34" width="0.254" layer="51"/>
-<wire x1="30.48" y1="53.34" x2="0" y2="53.34" width="0.254" layer="51"/>
-<wire x1="0" y1="53.34" x2="0" y2="46.99" width="0.254" layer="51"/>
-<wire x1="30.48" y1="1.778" x2="28.702" y2="0" width="0.1524" layer="20" curve="-90"/>
-<wire x1="1.778" y1="0" x2="0" y2="1.778" width="0.1524" layer="20" curve="-90"/>
-<wire x1="0" y1="42.672" x2="1.778" y2="44.45" width="0.1524" layer="20" curve="-90"/>
-<wire x1="28.702" y1="44.45" x2="30.48" y2="42.672" width="0.1524" layer="20" curve="-90"/>
-<text x="15.24" y="53.975" size="1.27" layer="51" align="bottom-center">Max Board Length</text>
-<dimension x1="28.575" y1="1.905" x2="1.905" y2="1.905" x3="15.24" y3="-2.54" textsize="1.27" textratio="10" layer="51" dtype="horizontal" unit="inch"/>
-<dimension x1="30.48" y1="1.728" x2="0" y2="2.54" x3="15.24" y3="-5.08" textsize="1.27" textratio="10" layer="51" dtype="horizontal" unit="inch"/>
-<dimension x1="1.905" y1="42.545" x2="1.905" y2="1.905" x3="35.56" y3="22.225" textsize="1.27" textratio="10" layer="51" dtype="vertical" unit="inch"/>
-<dimension x1="1.778" y1="44.45" x2="5.08" y2="0" x3="38.1" y3="22.225" textsize="1.27" textratio="10" layer="51" dtype="vertical" unit="inch"/>
-<dimension x1="0" y1="53.34" x2="2.54" y2="0" x3="40.64" y3="26.67" textsize="1.27" textratio="10" layer="51" dtype="vertical" unit="inch"/>
-<rectangle x1="22.098" y1="26.162" x2="30.48" y2="44.45" layer="42" rot="R180"/>
-<rectangle x1="22.098" y1="26.162" x2="30.48" y2="44.45" layer="41" rot="R180"/>
-<dimension x1="1.905" y1="42.545" x2="0.5579625" y2="43.8920375" x3="-5.07986875" y3="49.285071875" textsize="1.27" textratio="10" layer="51" dtype="radius" unit="inch"/>
-<dimension x1="29.28210625" y1="41.83789375" x2="27.86789375" y2="43.25210625" x3="34.925" y3="48.895" textsize="1.27" textratio="10" layer="51" dtype="diameter" visible="yes"/>
 <text x="30.099" y="3.81" size="1.016" layer="1" font="vector" ratio="15" rot="R90">v01</text>
-<text x="33.02" y="-3.81" size="1.778" layer="51">Note: Units are in Inches</text>
 <text x="29.464" y="6.096" size="1.016" layer="22" font="vector" ratio="15" rot="SMR270" align="center">4xM2.0</text>
-<text x="29.972" y="40.386" size="1.27" layer="22" font="vector" ratio="15" rot="SMR270">Name of Block</text>
+<wire x1="2.794" y1="39.37" x2="44.45" y2="39.37" width="0.4064" layer="20"/>
+<wire x1="44.45" y1="39.37" x2="44.45" y2="3.81" width="0.4064" layer="20"/>
+<wire x1="44.45" y1="3.81" x2="2.794" y2="3.81" width="0.4064" layer="20"/>
+<wire x1="2.794" y1="3.81" x2="2.794" y2="39.37" width="0.4064" layer="20"/>
 </plain>
 <attributes>
@@
 <pass name="Default">
 <param name="RoutingGrid" value="50mil"/>
+<param name="AutoGrid" value="1"/>
+<param name="Efforts" value="0"/>
+<param name="TopRouterVariant" value="1"/>
 <param name="tpViaShape" value="round"/>
 <param name="PrefDir.1" value="|"/>
@@
 </autorouter>
 <elements>
-<element name="FRAME1" library="SparkFun-Aesthetics" package="CREATIVE_COMMONS" value="FRAME-LETTER" x="-1.27" y="-13.97"/>
-<element name="LOGO2" library="SparkFun-Aesthetics" package="OSHW-LOGO-S" value="OSHW-LOGOS" x="5.842" y="1.778" rot="MR0"/>
-<element name="LOGO3" library="SparkFun-Aesthetics" package="SFE_LOGO_NAME_FLAME_.1" value="SFE_LOGO_NAME_FLAME.1_INCH" x="21.125003125" y="0.254" locked="yes" rot="MR0"/>
 <element name="J1" library="Edison" package="EDISON_DAUGHTER" value="EDISON_CONNECTOR_FULLMOUNTING_HOLES" x="27.94" y="3.81" locked="yes" rot="MR0"/>
 <element name="J2" library="Edison" package="DF40C-70DP-0.4(51)" value="EDISON_CONNECTOR_FULLHEADER" x="24.64" y="16.1798" locked="yes" rot="MR90"/>
-<element name="LOGO1" library="SparkFun-Aesthetics" package="OSHW-LOGO-S" value="OSHW-LOGOS" x="5.842" y="1.778" locked="yes"/>
-<element name="LOGO4" library="SparkFun-Aesthetics" package="SFE_LOGO_NAME_FLAME_.1" value="SFE_LOGO_NAME_FLAME.1_INCH" x="9.354996875" y="0.254" locked="yes"/>
-<element name="FID1" library="SparkFun-Aesthetics" package="FIDUCIAL-1X2" value="FIDUCIAL1X2" x="1.27" y="5.08" locked="yes"/>
-<element name="FID2" library="SparkFun-Aesthetics" package="FIDUCIAL-1X2" value="FIDUCIAL1X2" x="25.4" y="43.18" locked="yes"/>
-<element name="FID3" library="SparkFun-Aesthetics" package="FIDUCIAL-1X2" value="FIDUCIAL1X2" x="1.27" y="5.08" locked="yes" rot="MR0"/>
-<element name="FID4" library="SparkFun-Aesthetics" package="FIDUCIAL-1X2" value="FIDUCIAL1X2" x="25.4" y="43.18" locked="yes" rot="MR0"/>
 </elements>
 <signals>
 <signal name="GND">
 <polygon width="0.1778" layer="16" spacing="0.254" rank="6">
-<vertex x="30.48" y="42.672"/>
-<vertex x="30.48" y="1.778" curve="-90"/>
-<vertex x="28.702" y="0"/>
-<vertex x="1.778" y="0" curve="-90"/>
-<vertex x="0" y="1.778"/>
-<vertex x="0" y="42.672" curve="-90"/>
-<vertex x="1.778" y="44.45"/>
-<vertex x="28.702" y="44.45" curve="-90"/>
+<vertex x="44.45" y="38.1"/>
+<vertex x="44.45" y="5.08" curve="-90"/>
+<vertex x="43.18" y="3.81"/>
+<vertex x="4.064" y="3.81" curve="-90"/>
+<vertex x="2.794" y="5.08"/>
+<vertex x="2.794" y="38.1" curve="-90"/>
+<vertex x="4.064" y="39.37"/>
+<vertex x="43.18" y="39.37" curve="-90"/>
 </polygon>
 <polygon width="0.1778" layer="1" spacing="0.254" rank="6">
-<vertex x="30.48" y="1.778" curve="-90"/>
-<vertex x="28.752" y="0"/>
-<vertex x="1.778" y="0" curve="-90"/>
-<vertex x="0" y="1.778"/>
-<vertex x="0" y="42.672" curve="-90"/>
-<vertex x="1.778" y="44.45"/>
-<vertex x="28.702" y="44.45" curve="-90"/>
-<vertex x="30.48" y="42.672"/>
+<vertex x="44.45" y="5.334" curve="-90"/>
+<vertex x="43.23" y="3.81"/>
+<vertex x="4.064" y="3.81" curve="-90"/>
+<vertex x="2.794" y="4.826"/>
+<vertex x="2.794" y="38.1" curve="-90"/>
+<vertex x="4.064" y="39.37"/>
+<vertex x="43.18" y="39.37" curve="-90"/>
+<vertex x="44.45" y="38.1"/>
 </polygon>
 <via x="28.2448" y="22.1742" extent="1-16" drill="0.3302"/>
