File: Hardware/Block_Template.brd (EAGLE design)
At the start: 41.7 x 35.6 mm, 2 parts, among them J1 EDISON_CONNECTOR_FULLMOUNTING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, J2 EDISON_CONNECTOR_FULLHEADER

Commit message: nets defined, need final decision on connector
Parts:
- added R1: DNP, rcl:R0402
- added U$1: RIBBON_CONN_70_POS, kinetic:RIBBON_CONN_70_POS
Connections:
- new net N$2: R1.2, U$1.P$2, U$1.P$4, U$1.P$6
- net 1.8V: now also U$1.P$12
- net 3.3V: now also U$1.P$10, U$1.P$8
- net DCIN: now also U$1.P$14
- net FAULT: now also U$1.P$19
- net FW_RCVR: now also U$1.P$69
- net GND: now also U$1.P$1, U$1.P$11, U$1.P$13, U$1.P$15, U$1.P$5, U$1.P$9
- net GP109_SPI_2_CLK: now also U$1.P$55
- net GP110_SPI_2_FS0: now also U$1.P$53
- net GP111_SPI_2_FS1: now also U$1.P$51
- net GP114_SPI_2_RXD: now also U$1.P$59
- net GP115_SPI_2_TXD: now also U$1.P$57
- net GP128_UART_1_CTS: now also U$1.P$65
- net GP129_UART_1_RTS: now also U$1.P$63
- net GP12_PWM0: now also U$1.P$35
- net GP130_UART_1_RX: now also U$1.P$61
- net GP131_UART_1_TX: now also U$1.P$46
- net GP134_UART_2_RX: now also U$1.P$22
- net GP135_UART_2_TX: now also U$1.P$27
- net GP13_PWM1: now also U$1.P$33
- net GP14: now also U$1.P$48
- net GP15: now also U$1.P$42
- net GP165: now also U$1.P$25
- net GP182_PWM2: now also U$1.P$37
- net GP183_PWM3: now also U$1.P$39
- net GP19_I2C_1_SCL: now also U$1.P$41
- net GP20_I2C_1_SDA: now also U$1.P$43
- net GP27_I2C_6_SCL: now also U$1.P$45
- net GP28_I2C_6_SDA: now also U$1.P$47
- net GP40_I2S_2_CLK: now also U$1.P$52
- net GP41_I2S_2_FS: now also U$1.P$54
- net GP42_I2S_2_RXD: now also U$1.P$50
- net GP43_I2S_2_TXD: now also U$1.P$56
- net GP44: now also U$1.P$24
- net GP45: now also U$1.P$26
- net GP46: now also U$1.P$28
- net GP47: now also U$1.P$30
- net GP48: now also U$1.P$32
- net GP49: now also U$1.P$34
- net GP77_SD_0_CD#: now also U$1.P$60
- net GP78_SD_0_CLK: now also U$1.P$58
- net GP79_SD_0_CMD: now also U$1.P$62
- net GP80_SD_0_DAT0: now also U$1.P$66
- net GP81_SD_0_DAT1: now also U$1.P$70
- net GP82_SD_0_DAT2: now also U$1.P$64
- net GP83_SD_0_DAT3: now also U$1.P$68
- net GP84_SD_CLK_FB: now also U$1.P$44
- net MSIC_SLP_CLK: now also U$1.P$7
- net OSC_CLK_OUT: now also U$1.P$67
- net PSW: now also U$1.P$21
- net PWRBTN#: now also U$1.P$17
- net RCVR_MODE: now also U$1.P$31
- net RESET_OUT#: now also U$1.P$36
- net USB_DN: now also U$1.P$18
- net USB_DP: now also U$1.P$16
- net USB_ID: now also U$1.P$3
- net USB_VBUS: now also U$1.P$20
- net VSYS: now also R1.1
- net V_BAT_BKUP: now also U$1.P$23

Commit message: ready for manufacture
Parts:
- moved U$1 28.1 mm to (28.6, 48.0), flipped to the top, turned to 0 degrees
- moved R1 19.1 mm to (28.6, 43.7), turned to 180 degrees
- moved J2 9.09 mm to (32.9, 12.4)
- moved J1 9.09 mm to (36.2, 0.00)
Routing:
- net FW_RCVR: track 4.20 -> 100.5 mm
- net OSC_CLK_OUT: track 5.19 -> 99.3 mm
- net GP81_SD_0_DAT1: track 4.68 -> 97.2 mm
- net GP128_UART_1_CTS: track 4.68 -> 96.8 mm
- net GP80_SD_0_DAT0: track 5.27 -> 95.2 mm
- net GP83_SD_0_DAT3: track 5.27 -> 94.7 mm
- net GP129_UART_1_RTS: track 6.86 -> 94.1 mm
- net GP82_SD_0_DAT2: track 7.36 -> 93.3 mm
- net GP130_UART_1_RX: track 4.30 -> 89.4 mm
- net GP79_SD_0_CMD: track 8.08 -> 90.9 mm
- net GP43_I2S_2_TXD: track 8.31 -> 89.8 mm
- net GP114_SPI_2_RXD: track 6.38 -> 86.8 mm
- net GP115_SPI_2_TXD: track 8.10 -> 87.6 mm
- net GP77_SD_0_CD#: track 5.45 -> 83.0 mm
- net GP109_SPI_2_CLK: track 9.36 -> 86.8 mm
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- removed copper zone on layer 1, net VSYS
- removed copper zone on layer 16, net VSYS
Other:
- board size 41.7 x 35.6 mm -> 56.6 x 54.6 mm
- board text added: "BRIDGE FOR VSYS"
- board text removed: "4xM2.0"
- board text removed: "v01"

Commit message: off to fab.
Routing:
- net GP78_SD_0_CLK: track 81.9 -> 79.7 mm
- net GP183_PWM3: track 67.9 -> 66.1 mm
- net GP40_I2S_2_CLK: track 82.1 -> 83.1 mm
- net GP81_SD_0_DAT1: track 97.2 -> 98.2 mm
- net GP135_UART_2_TX: track 54.7 -> 54.0 mm
- net GP80_SD_0_DAT0: track 95.2 -> 95.9 mm
- net GP77_SD_0_CD#: track 83.0 -> 83.7 mm
- net GP44: track 50.5 -> 51.2 mm
- net FAULT: track 47.8 -> 47.3 mm
- net GP82_SD_0_DAT2: track 93.3 -> 93.9 mm
