File: Hardware/Block_Template.sch (EAGLE design)
At the start: 9 parts, among them J1 EDISON_CONNECTOR_FULLMOUNTING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, J2 EDISON_CONNECTOR_FULLHEADER

Commit message: initial cut
Parts:
- removed FID1, FID2, FID3, FID4: FIDUCIAL1X2, SparkFun-Aesthetics:FIDUCIAL1X2
- removed FRAME1: FRAME-LETTER, SparkFun-Aesthetics:FRAME-LETTER
- removed LOGO1: OSHW-LOGOS, SparkFun-Aesthetics:OSHW-LOGOS
- removed LOGO4: SFE_LOGO_NAME_FLAME.1_INCH, SparkFun-Aesthetics:SFE_LOGO_NAME_FLAME.1_INCH
Changed lines of the file:
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@@
 <?xml version="1.0" encoding="utf-8"?>
 <!DOCTYPE eagle SYSTEM "eagle.dtd">
-<eagle version="6.5.0">
+<eagle version="7.3.0">
 <drawing>
 <settings>
@@
 </classes>
 <parts>
-<part name="FRAME1" library="SparkFun-Aesthetics" deviceset="FRAME-LETTER" device=""/>
-<part name="LOGO1" library="SparkFun-Aesthetics" deviceset="OSHW-LOGO" device="S"/>
-<part name="LOGO4" library="SparkFun-Aesthetics" deviceset="SFE_LOGO_NAME_FLAME" device=".1_INCH"/>
 <part name="J1" library="Edison" deviceset="EDISON_CONNECTOR_FULL" device="MOUNTING_HOLES"/>
 <part name="GND3" library="supply1" deviceset="GND" device=""/>
 <part name="J2" library="Edison" deviceset="EDISON_CONNECTOR_FULL" device="HEADER" value="EDISON_CONNECTOR_FULLHEADER"/>
 <part name="GND4" library="supply1" deviceset="GND" device=""/>
-<part name="FID1" library="SparkFun-Aesthetics" deviceset="FIDUCIAL" device="1X2"/>
-<part name="FID2" library="SparkFun-Aesthetics" deviceset="FIDUCIAL" device="1X2"/>
-<part name="FID3" library="SparkFun-Aesthetics" deviceset="FIDUCIAL" device="1X2"/>
-<part name="FID4" library="SparkFun-Aesthetics" deviceset="FIDUCIAL" device="1X2"/>
 </parts>
 <sheets>
@@
 </plain>
 <instances>
-<instance part="FRAME1" gate="G$1" x="0" y="0"/>
-<instance part="FRAME1" gate="G$2" x="147.32" y="0"/>
-<instance part="LOGO1" gate="G$1" x="73.66" y="12.7"/>
-<instance part="LOGO4" gate="G$1" x="88.9" y="2.54"/>
-<instance part="FID1" gate="G$1" x="246.38" y="25.4"/>
-<instance part="FID2" gate="G$1" x="241.3" y="25.4"/>
-<instance part="FID3" gate="G$1" x="246.38" y="30.48"/>
-<instance part="FID4" gate="G$1" x="241.3" y="30.48"/>
 </instances>
 <busses>
