File: Hardware/Block_Template.sch (EAGLE design)
At the start: 2 parts, among them J1 EDISON_CONNECTOR_FULLMOUNTING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, J2 EDISON_CONNECTOR_FULLHEADER

Commit message: nets defined, need final decision on connector
Parts:
- added R1: DNP, rcl:R-US_R0402
- added U$1: RIBBON_CONN_70_POS, kinetic:RIBBON_CONN_70_POS
Connections:
- new net N$2: R1.2, U$1.VSYS@1, U$1.VSYS@2, U$1.VSYS@3
- net 1.8V: now also U$1.1.8V
- net 3.3V: now also U$1.3.3V@1, U$1.3.3V@2
- net DCIN: now also U$1.DCIN
- net FAULT: now also U$1.FAULT
- net FW_RCVR: now also U$1.FW_RCVR
- net GND: now also U$1.GND@1, U$1.GND@2, U$1.GND@3, U$1.GND@4, U$1.GND@5, U$1.GND@6
- net GP109_SPI_2_CLK: now also U$1.GP109_SPI_2_CLK
- net GP110_SPI_2_FS0: now also U$1.GP110_SPI_2_FS0
- net GP111_SPI_2_FS1: now also U$1.GP111_SPI_2_FS1
- net GP114_SPI_2_RXD: now also U$1.GP114_SPI_2_RXD
- net GP115_SPI_2_TXD: now also U$1.GP115_SPI_2_TXD
- net GP128_UART_1_CTS: now also U$1.GP128_UART_1_CTS
- net GP129_UART_1_RTS: now also U$1.GP129_UART_1_RTS
- net GP12_PWM0: now also U$1.GP12_PWM0
- net GP130_UART_1_RX: now also U$1.GP130_UART_1_RX
- net GP131_UART_1_TX: now also U$1.GP131_UART_1_TX
- net GP134_UART_2_RX: now also U$1.GP134_UART_2_RX
- net GP135_UART_2_TX: now also U$1.GP135_UART_2_TX
- net GP13_PWM1: now also U$1.GP13_PWM1
- net GP14: now also U$1.GP14
- net GP15: now also U$1.GP15
- net GP165: now also U$1.GP165
- net GP182_PWM2: now also U$1.GP182_PWM2
- net GP183_PWM3: now also U$1.GP183_PWM3
- net GP19_I2C_1_SCL: now also U$1.GP19_I2C_1_SCL
- net GP20_I2C_1_SDA: now also U$1.GP20_I2C_1_SDA
- net GP27_I2C_6_SCL: now also U$1.GP27_I2C_6_SCL
- net GP28_I2C_6_SDA: now also U$1.GP28_I2C_6_SDA
- net GP40_I2S_2_CLK: now also U$1.GP40_I2S_2_CLK
- net GP41_I2S_2_FS: now also U$1.GP41_I2S_2_FS
- net GP42_I2S_2_RXD: now also U$1.GP42_I2S_2_RXD
- net GP43_I2S_2_TXD: now also U$1.GP43_I2S_2_TXD
- net GP44: now also U$1.GP44
- net GP45: now also U$1.GP45
- net GP46: now also U$1.GP46
- net GP47: now also U$1.GP47
- net GP48: now also U$1.GP48
- net GP49: now also U$1.GP49
- net GP77_SD_0_CD#: now also U$1.GP77_SD_0_CD#
- net GP78_SD_0_CLK: now also U$1.GP78_SD_0_CLK
- net GP79_SD_0_CMD: now also U$1.GP79_SD_0_CMD
- net GP80_SD_0_DAT0: now also U$1.GP80_SD_0_DAT0
- net GP81_SD_0_DAT1: now also U$1.GP81_SD_0_DAT1
- net GP82_SD_0_DAT2: now also U$1.GP82_SD_0_DAT2
- net GP83_SD_0_DAT3: now also U$1.GP83_SD_0_DAT3
- net GP84_SD_CLK_FB: now also U$1.GP84_SD_CLK_FB
- net MSIC_SLP_CLK: now also U$1.MSIC_SLP_CLK
- net OSC_CLK_OUT: now also U$1.OSC_CLK_OUT_0
- net PSW: now also U$1.PSW
- net PWRBTN#: now also U$1.PWRBTN#
- net RCVR_MODE: now also U$1.RCVR_MODE
- net RESET_OUT#: now also U$1.RESET_OUT#
- net USB_DN: now also U$1.USB_DN
- net USB_DP: now also U$1.USB_DP
- net USB_ID: now also U$1.USB_ID
- net USB_VBUS: now also U$1.USB_VBUS
- net VSYS: now also R1.1
- net V_BAT_BKUP: now also U$1.V_VAT_BKUP
